File: hw/irq.kicad_sch (KiCad schematic)
At the start: 8 parts, among them U1 74LS85, U11 74ACT00P, U18 74LS148, U2 74HCT574, U20 74HCT574, U5 74AHCT02, U8 74AS04N

Commit message: add hw design for veraduino
Other:
- moved on the sheet: U11B, U5A, U5C, U8E

Commit message: clean up hw schematics
Changed lines of the file:
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@@
+    (stroke (width 0) (type default))
+  )
+  (wire (pts (xy 27.94 133.35) (xy 27.94 132.08))
     (stroke (width 0) (type default))
   )
@@
     )
   )
-  (symbol (lib_id "power:Earth") (at 27.94 132.08 0) (unit 1)
+  (symbol (lib_id "power:Earth") (at 27.94 133.35 0) (unit 1)
     (in_bom yes) (on_board yes) (dnp no) (fields_autoplaced)
-    (property "Reference" "#PWR035" (at 27.94 138.43 0)
-      (effects (font (size 1.27 1.27)) hide)
-    )
-    (property "Value" "Earth" (at 27.94 135.89 0)
-      (effects (font (size 1.27 1.27)) hide)
-    )
-    (property "Footprint" "" (at 27.94 132.08 0)
-      (effects (font (size 1.27 1.27)) hide)
-    )
-    (property "Datasheet" "~" (at 27.94 132.08 0)
-      (effects (font (size 1.27 1.27)) hide)
-    )
+    (property "Reference" "#PWR035" (at 27.94 139.7 0)
+      (effects (font (size 1.27 1.27)) hide)
+    )
+    (property "Value" "Earth" (at 27.94 137.16 0)
+      (effects (font (size 1.27 1.27)) hide)
+    )
+    (property "Footprint" "" (at 27.94 133.35 0)
+      (effects (font (size 1.27 1.27)) hide)
+    )
+    (property "Datasheet" "~" (at 27.94 133.35 0)
+      (effects (font (size 1.27 1.27)) hide)
+    )
